File: pcb/keyboard/v0.1/keyboard.kicad_sch (KiCad schematic)
At the start: 139 parts, among them J1 USB2.0, J2 SWD, SW1 BACKTICK, SW10 9, SW11 0, SW12 BACKSPACE, SW13 TAB, SW14 Q, SW15 W, SW16 E, SW17 R, SW18 T, SW19 Y, SW2 1, SW20 U, SW21 I, SW22 O, SW23 P, SW24 RETURN, SW25 CAPS, SW26 A, SW27 S, SW28 D, SW29 F, SW3 2, SW30 G, SW31 H, SW32 J, SW33 K, SW34 L, SW35 SEMI, SW36 QUOTE, SW37 LSHIFT, SW38 Z, SW39 X, SW4 3, SW40 C, SW41 V, SW42 B, SW43 N, SW44 M, SW45 COMMA, SW46 DOT, SW47 QUEST, SW48 RSHIFT, SW49 FN, SW5 4, SW50 LCTRL, SW51 LSUPER, SW52 LALT, SW53 SPACE, SW54 RALT, SW55 RSUPER, SW56 MENU, SW57 RCTRL, SW59 C2, SW6 5, SW60 C3, SW61 C4, SW62 C5, SW7 6, SW8 7, SW9 8, U1 MDBT50Q-P1MV2, Y1 32.768

Commit message: Complete redesign of the keyboard module
Parts:
- removed D10, D11, D12, D3, D4, D5, D53, D6, D60, D61, D7, D8, D9: 1N4148, Diode_SMD:D_SOD-523, symbol Device:D
- removed SW10: 9, TH-A1OC:tact_switch_4.5x4.5_PTS647, symbol TH-A10C:SW_Push_45deg
- removed SW11: 0, TH-A1OC:tact_switch_4.5x4.5_PTS647, symbol TH-A10C:SW_Push_45deg
- removed SW12: BACKSPACE, TH-A1OC:tact_switch_4.5x4.5_PTS647, symbol TH-A10C:SW_Push_45deg
- removed SW3: 2, TH-A1OC:tact_switch_4.5x4.5_PTS647, symbol TH-A10C:SW_Push_45deg
- removed SW4: 3, TH-A1OC:tact_switch_4.5x4.5_PTS647, symbol TH-A10C:SW_Push_45deg
- removed SW5: 4, TH-A1OC:tact_switch_4.5x4.5_PTS647, symbol TH-A10C:SW_Push_45deg
- removed SW53: SPACE, TH-A1OC:tact_switch_4.5x4.5_PTS647, symbol TH-A10C:SW_Push_45deg
- removed SW6: 5, TH-A1OC:tact_switch_4.5x4.5_PTS647, symbol TH-A10C:SW_Push_45deg
- removed SW60: C3, TH-A1OC:tact_switch_4.5x4.5_PTS647, symbol TH-A10C:SW_Push_45deg
- removed SW61: C4, TH-A1OC:tact_switch_4.5x4.5_PTS647, symbol TH-A10C:SW_Push_45deg
- removed SW7: 6, TH-A1OC:tact_switch_4.5x4.5_PTS647, symbol TH-A10C:SW_Push_45deg
- removed SW8: 7, TH-A1OC:tact_switch_4.5x4.5_PTS647, symbol TH-A10C:SW_Push_45deg
- removed SW9: 8, TH-A1OC:tact_switch_4.5x4.5_PTS647, symbol TH-A10C:SW_Push_45deg
- SW1: value BACKTICK -> SPACE
- SW2: value 1 -> SPACE
Connections:
- net INPUT1: no longer D1.1 (K)
- net INPUT2: no longer D2.1 (K)
- net INPUT5: now also D1.1 (K)
- net INPUT8: now also D2.1 (K)
- net SOURCE1: now also SW13.1, SW14.1, SW15.1, SW16.1, SW17.1, SW18.1, SW19.1, SW20.1, SW21.1, SW22.1, SW23.1, SW24.1, U1.21 (P0.05/AIN3); no longer SW1.1, SW2.1, U1.19 (P0.26)
- net SOURCE2: now also SW25.1, SW26.1, SW27.1, SW28.1, SW29.1, SW30.1, SW31.1, SW32.1, SW33.1, SW34.1, SW35.1, SW36.1, U1.23 (P0.07/TRACECLK); no longer SW13.1, SW14.1, SW15.1, SW16.1, SW17.1, SW18.1, SW19.1, SW20.1, SW21.1, SW22.1, SW23.1, SW24.1, U1.20 (P0.04/AIN2)
- net SOURCE3: now also SW37.1, SW38.1, SW39.1, SW40.1, SW41.1, SW42.1, SW43.1, SW44.1, SW45.1, SW46.1, SW47.1, SW48.1, U1.25 (P1.08); no longer SW25.1, SW26.1, SW27.1, SW28.1, SW29.1, SW30.1, SW31.1, SW32.1, SW33.1, SW34.1, SW35.1, SW36.1, U1.21 (P0.05/AIN3)
- net SOURCE4: now also SW1.1, SW2.1, SW49.1, SW50.1, SW51.1, SW52.1, SW54.1, SW55.1, SW56.1, SW57.1, U1.27 (P0.11/TRACEDATA2); no longer SW37.1, SW38.1, SW39.1, SW40.1, SW41.1, SW42.1, SW43.1, SW44.1, SW45.1, SW46.1, SW47.1, SW48.1, U1.22 (P0.06)
- net SOURCE5: now also SW59.1, SW62.1, U1.29 (P0.12/TRACEDATA1); no longer SW49.1, SW50.1, SW51.1, SW52.1, SW54.1, SW55.1, SW56.1, SW57.1, U1.23 (P0.07/TRACECLK)
- removed net SOURCE6: SW59.1, SW62.1, U1.24 (P0.08)
- no-connect marks 26 -> 27
