File: pcb/keyboard/v0.1/keyboard.kicad_pcb (KiCad board)
At the start: 4 copper layers, 80.8 x 67.2 mm, 139 parts, among them J1 USB2.0, J2 SWD, SW1 BACKTICK, SW10 9, SW11 0, SW12 BACKSPACE, SW13 TAB, SW14 Q, SW15 W, SW16 E, SW17 R, SW18 T, SW19 Y, SW2 1, SW20 U, SW21 I, SW22 O, SW23 P, SW24 RETURN, SW25 CAPS, SW26 A, SW27 S, SW28 D, SW29 F, SW3 2, SW30 G, SW31 H, SW32 J, SW33 K, SW34 L, SW35 SEMI, SW36 QUOTE, SW37 LSHIFT, SW38 Z, SW39 X, SW4 3, SW40 C, SW41 V, SW42 B, SW43 N, SW44 M, SW45 COMMA, SW46 DOT, SW47 QUEST, SW48 RSHIFT, SW49 FN, SW5 4, SW50 LCTRL, SW51 LSUPER, SW52 LALT, SW53 SPACE, SW54 RALT, SW55 RSUPER, SW56 MENU, SW57 RCTRL, SW59 C2, SW6 5, SW60 C3, SW61 C4, SW62 C5, SW7 6, SW8 7, SW9 8, U1 MDBT50Q-P1MV2, Y1 32.768

Commit message: Complete redesign of the keyboard module
Parts:
- removed D10, D11, D12, D3, D4, D5, D53, D6, D60, D61, D7, D8, D9: 1N4148, Diode_SMD:D_SOD-523
- removed SW10: 9, TH-A1OC:tact_switch_4.5x4.5_PTS647
- removed SW11: 0, TH-A1OC:tact_switch_4.5x4.5_PTS647
- removed SW12: BACKSPACE, TH-A1OC:tact_switch_4.5x4.5_PTS647
- removed SW3: 2, TH-A1OC:tact_switch_4.5x4.5_PTS647
- removed SW4: 3, TH-A1OC:tact_switch_4.5x4.5_PTS647
- removed SW5: 4, TH-A1OC:tact_switch_4.5x4.5_PTS647
- removed SW53: SPACE, TH-A1OC:tact_switch_4.5x4.5_PTS647
- removed SW6: 5, TH-A1OC:tact_switch_4.5x4.5_PTS647
- removed SW60: C3, TH-A1OC:tact_switch_4.5x4.5_PTS647
- removed SW61: C4, TH-A1OC:tact_switch_4.5x4.5_PTS647
- removed SW7: 6, TH-A1OC:tact_switch_4.5x4.5_PTS647
- removed SW8: 7, TH-A1OC:tact_switch_4.5x4.5_PTS647
- removed SW9: 8, TH-A1OC:tact_switch_4.5x4.5_PTS647
- SW1: value BACKTICK -> SPACE
- SW2: value 1 -> SPACE
- moved SW62 152.9 mm to (-22.8, 119.5)
- moved SW59 85.6 mm to (-22.5, 113.3)
- moved J1 57.3 mm to (132.5, 89.3), turned to 0 degrees
- moved J2 54.5 mm to (132.5, 92.4), turned to 0 degrees
- moved C1 52.2 mm to (133.1, 95.5), turned to 0 degrees
- moved C2 51.1 mm to (133.1, 98.5), turned to 0 degrees
- moved Y1 50.0 mm to (137.9, 95.7)
- moved JP1 49.9 mm to (137.5, 99.1), turned to 0 degrees
- moved R3 47.5 mm to (124.8, 101.5), turned to 0 degrees
- moved R1 46.9 mm to (124.8, 96.5)
- moved R2 46.4 mm to (124.8, 99.0), turned to 0 degrees
- moved R4 44.2 mm to (124.8, 104.0)
- moved TP2 43.9 mm to (128.9, 93.8), turned to 0 degrees
- moved L1 41.6 mm to (124.8, 94.0)
- moved D62 40.0 mm to (92.7, 102.5)
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Connections:
- D1 pad 1: /INPUT1 -> /INPUT5
- D2 pad 1: /INPUT2 -> /INPUT8
- SW1 pad 1: /SOURCE1 -> /SOURCE4
- SW13 pad 1: /SOURCE2 -> /SOURCE1
- SW14 pad 1: /SOURCE2 -> /SOURCE1
- SW15 pad 1: /SOURCE2 -> /SOURCE1
- SW16 pad 1: /SOURCE2 -> /SOURCE1
- SW17 pad 1: /SOURCE2 -> /SOURCE1
- SW18 pad 1: /SOURCE2 -> /SOURCE1
- SW19 pad 1: /SOURCE2 -> /SOURCE1
- SW2 pad 1: /SOURCE1 -> /SOURCE4
- SW20 pad 1: /SOURCE2 -> /SOURCE1
- SW21 pad 1: /SOURCE2 -> /SOURCE1
- SW22 pad 1: /SOURCE2 -> /SOURCE1
- SW23 pad 1: /SOURCE2 -> /SOURCE1
- SW24 pad 1: /SOURCE2 -> /SOURCE1
- SW25 pad 1: /SOURCE3 -> /SOURCE2
- SW26 pad 1: /SOURCE3 -> /SOURCE2
- SW27 pad 1: /SOURCE3 -> /SOURCE2
- SW28 pad 1: /SOURCE3 -> /SOURCE2
- SW29 pad 1: /SOURCE3 -> /SOURCE2
- SW30 pad 1: /SOURCE3 -> /SOURCE2
- SW31 pad 1: /SOURCE3 -> /SOURCE2
- SW32 pad 1: /SOURCE3 -> /SOURCE2
- SW33 pad 1: /SOURCE3 -> /SOURCE2
- SW34 pad 1: /SOURCE3 -> /SOURCE2
- SW35 pad 1: /SOURCE3 -> /SOURCE2
- SW36 pad 1: /SOURCE3 -> /SOURCE2
- SW37 pad 1: /SOURCE4 -> /SOURCE3
- SW38 pad 1: /SOURCE4 -> /SOURCE3
- SW39 pad 1: /SOURCE4 -> /SOURCE3
- SW40 pad 1: /SOURCE4 -> /SOURCE3
- SW41 pad 1: /SOURCE4 -> /SOURCE3
- SW42 pad 1: /SOURCE4 -> /SOURCE3
- SW43 pad 1: /SOURCE4 -> /SOURCE3
- SW44 pad 1: /SOURCE4 -> /SOURCE3
- SW45 pad 1: /SOURCE4 -> /SOURCE3
- SW46 pad 1: /SOURCE4 -> /SOURCE3
- SW47 pad 1: /SOURCE4 -> /SOURCE3
- SW48 pad 1: /SOURCE4 -> /SOURCE3
- SW49 pad 1: /SOURCE5 -> /SOURCE4
- SW50 pad 1: /SOURCE5 -> /SOURCE4
- SW51 pad 1: /SOURCE5 -> /SOURCE4
- SW52 pad 1: /SOURCE5 -> /SOURCE4
- SW54 pad 1: /SOURCE5 -> /SOURCE4
- SW55 pad 1: /SOURCE5 -> /SOURCE4
- SW56 pad 1: /SOURCE5 -> /SOURCE4
- SW57 pad 1: /SOURCE5 -> /SOURCE4
- SW59 pad 1: /SOURCE6 -> /SOURCE5
- SW62 pad 1: /SOURCE6 -> /SOURCE5
- U1 pad 19: /SOURCE1 -> unconnected-(U1A-P0.26-Pad19)
- U1 pad 20: /SOURCE2 -> unconnected-(U1A-P0.04/AIN2-Pad20)
- U1 pad 21: /SOURCE3 -> /SOURCE1
- U1 pad 22: /SOURCE4 -> unconnected-(U1A-P0.06-Pad22)
- U1 pad 23: /SOURCE5 -> /SOURCE2
- U1 pad 24: /SOURCE6 -> unconnected-(U1A-P0.08-Pad24)
- U1 pad 25: unconnected-(U1A-P1.08-Pad25) -> /SOURCE3
- U1 pad 27: unconnected-(U1A-P0.11/TRACEDATA2-Pad27) -> /SOURCE4
- U1 pad 29: unconnected-(U1A-P0.12/TRACEDATA1-Pad29) -> /SOURCE5
Routing:
- net /SOURCE1: track 162.5 -> 0.00 mm, vias 1 -> 0
- net /SOURCE3: track 161.7 -> 0.00 mm, vias 1 -> 0
- net /SOURCE4: track 161.2 -> 0.00 mm, vias 1 -> 0
- net /SOURCE2: track 146.4 -> 0.00 mm, vias 1 -> 0
- net /SOURCE5: track 138.9 -> 0.00 mm, vias 1 -> 0
- net Net-(D17-A): track 7.34 -> 0.00 mm
- net Net-(D16-A): track 7.34 -> 0.00 mm
- net Net-(D15-A): track 7.34 -> 0.00 mm
- net Net-(D14-A): track 7.34 -> 0.00 mm
- net Net-(D13-A): track 7.34 -> 0.00 mm
- net Net-(D21-A): track 7.34 -> 0.00 mm
- net Net-(D20-A): track 7.34 -> 0.00 mm
- net Net-(D19-A): track 7.34 -> 0.00 mm
- net Net-(D18-A): track 7.34 -> 0.00 mm
- net Net-(D49-A): track 7.32 -> 0.00 mm
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Other:
- board size 80.8 x 67.2 mm -> 80 x 51 mm
- board text removed: "VDD"
