File: pcb/v0.1/gpio.kicad_sch (KiCad schematic)
At the start: 29 parts, among them J5 Micro_SD_molex, J7 AudioJack3, SW1 SW_Push_45deg, U3 PCM5102A, U4 RT9742GGJ5

Commit message: Add high side switch to dac so its not draining power when pi is off
Parts:
- added C27, C28: 10uf, Capacitor_SMD:C_0805_2012Metric, symbol TH-1-CC:C_10uf
- added TP3: TestPoint, symbol Connector:TestPoint
- added U7: RT9742GGJ5, Package_TO_SOT_SMD:TSOT-23-5, symbol TH-1-CC:RT9742GGJ5
Connections:
- net +3v3_LDO: now also C28.2, U7.5 (VIN); no longer FB1.1, FB2.1, TP1.1
- net +3v3_PI: now also U7.4 (EN)
- net GND: now also C27.1, C28.1, U7.2 (GND)
- net SD_nFLAG: now reaches U4.3 (nFLAG)
- net SD_nFLAG: now also TP1.1
- new net: C27.2, FB1.1, FB2.1, U7.1 (VOUT)
- new net DAC_nFLAG: TP3.1, U7.3 (nFLAG)
- no-connect marks 3 -> 2
Other:
- note added: "NOTE: nFlag needs pullup if testing"
- note added: "RPI boot SD card"
- note removed: "Add High side switch so its not powered when the pi is off. +10uf cap at switch out"
- note removed: "CM5Lite SDCARD I/F"
- moved on the sheet: Module1A, TP1
