File: pcb/v0.1/mainboard.kicad_sch (KiCad schematic)
At the start: 15 parts, among them J1 Conn_01x02_Pin, J2 TYPE_C_Receptacle, J3 Conn_01x04_Pin, U1 AP2112K-3.3TRG1

Commit message: Rough layout for power, SD and audio
Added the rough layout for the power input USB port, the 3v3 regulator,
the micro SD card and the entire audio subsystem including the dac and
its high side switch.
Other:
- moved on the sheet: TP7
Changed lines of the file:
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@@
+	)
+	(junction
+		(at 67.31 38.1)
+		(diameter 0)
+		(color 0 0 0 0)
 	)
 	(junction
@@
 	(junction
 		(at 59.69 172.72)
-		(diameter 0)
-		(color 0 0 0 0)
-	)
-	(junction
-		(at 74.93 38.1)
 		(diameter 0)
 		(color 0 0 0 0)
@@
 	(wire
 		(pts
+			(xy 67.31 38.1) (xy 83.82 38.1)
+		)
+		(stroke
+			(width 0)
+			(type default)
+		)
+	)
+	(wire
+		(pts
 			(xy 274.32 148.59) (xy 274.32 161.29)
 		)
@@
 	(wire
 		(pts
-			(xy 74.93 38.1) (xy 83.82 38.1)
-		)
-		(stroke
-			(width 0)
-			(type default)
-		)
-	)
-	(wire
-		(pts
 			(xy 69.85 57.15) (xy 71.12 57.15)
 		)
@@
 	(wire
 		(pts
-			(xy 53.34 38.1) (xy 74.93 38.1)
+			(xy 53.34 38.1) (xy 67.31 38.1)
 		)
 		(stroke
@@
 	(symbol
 		(lib_id "Connector:TestPoint")
-		(at 74.93 38.1 0)
+		(at 67.31 38.1 0)
 		(unit 1)
 		(body_style 1)
@@
 		(dnp no)
 		(property "Reference" "TP7"
-			(at 73.66 34.544 0)
+			(at 66.04 34.544 0)
 			(show_name no)
 			(do_not_autoplace no)
@@
 		)
 		(property "Value" "TestPoint"
-			(at 72.39 33.5281 0)
+			(at 64.77 33.5281 0)
 			(hide yes)
 			(show_name no)
@@
 		)
 		(property "Footprint" "TestPoint:TestPoint_Pad_D1.0mm"
-			(at 80.01 38.1 0)
+			(at 72.39 38.1 0)
 			(hide yes)
 			(show_name no)
@@
 		)
 		(property "Datasheet" ""
-			(at 80.01 38.1 0)
+			(at 72.39 38.1 0)
 			(hide yes)
 			(show_name no)
@@
 		)
 		(property "Description" "test point"
-			(at 74.93 38.1 0)
+			(at 67.31 38.1 0)
 			(hide yes)
 			(show_name no)

Commit message: USB differential pairs complete.
Had to break these out from the rest of the pcb as they just didn't add
up otherwise. Will continue to do the high speed lines separately before
re assembling the pcb.
Parts:
- J2: footprint Connector_USB:USB_C_Receptacle_Molex_105450-0101 -> TH-1-CC_footprints:USB4056-03-A; Digikey Part no WM12856TR-ND -> 2073-USB4056-03-ATR-ND; Distributor Digikey https://www.digikey.co.uk/en/products/detail/molex/10545001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 -> https://www.digikey.co.uk/en/products/detail/gct/USB4056-03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; Manufacturer MOLEX -> GCT; Mfr. Part no 1054500101 -> USB4056-03-A
Changed lines of the file:
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@@
 			)
 		)
-		(property "Footprint" "Connector_USB:USB_C_Receptacle_Molex_105450-0101"
+		(property "Footprint" "TH-1-CC_footprints:USB4056-03-A"
 			(at 38.1 66.04 0)
 			(hide yes)
@@
 			)
 		)
-		(property "Datasheet" "https://www.molex.com/pdm_docs/ps/PS-105448-001.pdf"
+		(property "Datasheet" "https://gct.co/files/specs/usb4056-spec.pdf"
 			(at 38.1 66.04 0)
 			(hide yes)
@@
 			)
 		)
-		(property "Description" "USB Full-Featured Type-C Receptacle connector"
+		(property "Description" "USB Type-c 24pin 5A 48V"
 			(at 34.29 66.04 0)
 			(hide yes)
@@
 			)
 		)
-		(property "Manufacturer" "MOLEX"
+		(property "Manufacturer" "GCT"
 			(at 34.29 66.04 0)
 			(hide yes)
@@
 			)
 		)
-		(property "Mfr. Part no" "1054500101"
+		(property "Mfr. Part no" "USB4056-03-A"
 			(at 34.29 66.04 0)
 			(hide yes)
@@
 			)
 		)
-		(property "Distributor Digikey" "https://www.digikey.co.uk/en/products/detail/molex/1054500101/5843890"
+		(property "Distributor Digikey" "https://www.digikey.co.uk/en/products/detail/gct/USB4056-03-A/14638038?utm_source=oemsecrets&utm_medium=aggregator&utm_campaign=buynow"
 			(at 34.29 66.04 0)
 			(hide yes)
@@
 			)
 		)
-		(property "Digikey Part no" "WM12856TR-ND"
+		(property "Digikey Part no" "2073-USB4056-03-ATR-ND"
 			(at 34.29 66.04 0)
 			(hide yes)

Commit message: High power routing
Finished the single high power line. It should be able to hold peaks of
5A without heating up too much, but only testing will reveal.
Connections:
- net USB2_CC1: now also D5.1 (IO1); no longer D5.2 (IO2)
- net USB2_CC2: now also D5.2 (IO2); no longer D5.1 (IO1)
- net USB2_N: now also D4.1 (IO1); no longer D4.2 (IO2)
- net USB2_P: now also D4.2 (IO2); no longer D4.1 (IO1)
Changed lines of the file:
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@@
 		(lib_id "TH-1-CC:High_speed_TVS_array")
 		(at 64.77 45.72 90)
+		(mirror x)
 		(unit 1)
 		(body_style 1)
@@
 		(dnp no)
 		(property "Reference" "D5"
-			(at 60.96 40.386 90)
+			(at 61.468 39.878 90)
 			(show_name no)
 			(do_not_autoplace no)
@@
 		)
 		(property "Value" "TECH REPUBLIC ESD5302F"
-			(at 64.77 36.83 90)
+			(at 64.77 54.61 90)
 			(hide yes)
 			(show_name no)
@@
 		)
 		(property "Footprint" "Package_TO_SOT_SMD:SOT-23"
-			(at 72.39 32.512 0)
+			(at 72.39 58.928 0)
 			(hide yes)
 			(show_name no)
@@
 		)
 		(property "Datasheet" "https://www.lcsc.com/datasheet/C2841442.pdf?spm=wm.sxq.inf.ggs&lcsc_vid=QAILXlUCRldfUlcDQgANV1IDE1JYXwJWRANcAwFRRgAxVlNeRVdeVF1VT1JfUDsOAxUeFF5JWBYZEEoKFBINSQcJGk4NBhADEA4cHktRR1NADxALGw%3D%3D"
-			(at 80.01 -70.104 0)
+			(at 80.01 161.544 0)
 			(hide yes)
 			(show_name no)
@@
 		)
 		(property "Description" "ESD DIODE 5VWM 14VC SOT-23"
-			(at 74.93 18.796 0)
+			(at 74.93 72.644 0)
 			(hide yes)
 			(show_name no)
@@
 		)
 		(property "Manufacturer" "TECH PUBLIC"
-			(at 70.104 26.924 0)
+			(at 70.104 64.516 0)
 			(hide yes)
 			(show_name no)
@@
 		)
 		(property "Mfr. Part no." "ESD5302F"
-			(at 70.104 15.24 0)
+			(at 70.104 76.2 0)
 			(hide yes)
 			(show_name no)
@@
 		)
 		(property "Distributor LCSC" "https://www.lcsc.com/product-detail/C2841442.html?lcsc_vid=QAILXlUCRldfUlcDQgANV1IDE1JYXwJWRANcAwFRRgAxVlNeRVdeVF1VT1JfUDsOAxUeFF5JWBYZEEoKFBINSQcJGk4NBhADEA4cHktRR1NADxALGw%3D%3D"
-			(at 82.55 -63.246 0)
+			(at 82.55 154.686 0)
 			(hide yes)
 			(show_name no)
@@
 		)
 		(property "LCSC Part no." "C2841442"
-			(at 77.47 28.448 0)
+			(at 77.47 62.992 0)
 			(hide yes)
 			(show_name no)
@@
 		)
 		(property "Stock" "NO!"
-			(at 67.31 51.308 90)
+			(at 67.818 51.308 90)
 			(show_name no)
 			(do_not_autoplace no)
@@
 		(lib_id "TH-1-CC:High_speed_TVS_array")
 		(at 64.77 57.15 90)
+		(mirror x)
 		(unit 1)
 		(body_style 1)
@@
 		(dnp no)
 		(property "Reference" "D4"
-			(at 61.214 52.07 90)
+			(at 60.452 51.816 90)
 			(show_name no)
 			(do_not_autoplace no)
@@
 		)
 		(property "Value" "TECH REPUBLIC ESD5302F"
-			(at 64.77 48.26 90)
+			(at 64.77 66.04 90)
 			(hide yes)
 			(show_name no)
@@
 		)
 		(property "Footprint" "Package_TO_SOT_SMD:SOT-23"
-			(at 72.39 43.942 0)
+			(at 72.39 70.358 0)
 			(hide yes)
 			(show_name no)
@@
 		)
 		(property "Datasheet" "https://www.lcsc.com/datasheet/C2841442.pdf?spm=wm.sxq.inf.ggs&lcsc_vid=QAILXlUCRldfUlcDQgANV1IDE1JYXwJWRANcAwFRRgAxVlNeRVdeVF1VT1JfUDsOAxUeFF5JWBYZEEoKFBINSQcJGk4NBhADEA4cHktRR1NADxALGw%3D%3D"
-			(at 80.01 -58.674 0)
+			(at 80.01 172.974 0)
 			(hide yes)
 			(show_name no)
@@
 		)
 		(property "Description" "ESD DIODE 5VWM 14VC SOT-23"
-			(at 74.93 30.226 0)
+			(at 74.93 84.074 0)
 			(hide yes)
 			(show_name no)
@@
 		)
 		(property "Manufacturer" "TECH PUBLIC"
-			(at 70.104 38.354 0)
+			(at 70.104 75.946 0)
 			(hide yes)
 			(show_name no)
@@
 		)
 		(property "Mfr. Part no." "ESD5302F"
-			(at 70.104 26.67 0)
+			(at 70.104 87.63 0)
 			(hide yes)
 			(show_name no)
@@
 		)
 		(property "Distributor LCSC" "https://www.lcsc.com/product-detail/C2841442.html?lcsc_vid=QAILXlUCRldfUlcDQgANV1IDE1JYXwJWRANcAwFRRgAxVlNeRVdeVF1VT1JfUDsOAxUeFF5JWBYZEEoKFBINSQcJGk4NBhADEA4cHktRR1NADxALGw%3D%3D"
-			(at 82.55 -51.816 0)
+			(at 82.55 166.116 0)
 			(hide yes)
 			(show_name no)
@@
 		)
 		(property "LCSC Part no." "C2841442"
-			(at 77.47 39.878 0)
+			(at 77.47 74.422 0)
 			(hide yes)
 			(show_name no)
@@
 		)
 		(property "Stock" "NO!"
-			(at 67.818 62.738 90)
-			(show_name no)
-			(do_not_autoplace no)
+			(at 67.31 62.738 90)
+			(show_name no)
+			(do_not_autoplace no)

Commit message: A large chunk of the pcb routing + shrinking the board
Did a large chunk of the PCB routing, probably just under half of all
remaining traces. Additionally I shrank the pcb to below 100x100 as it
reduces the price of manufacturing by roughly 4x
Parts:
- added H1, H2, H3, H4: MountingHole_Pad, MountingHole:MountingHole_2.2mm_M2_DIN965_Pad, symbol Mechanical:MountingHole_Pad
Connections:
- net GND: now also H1.1, H2.1, H3.1, H4.1
- net USB2_CC1: now also D5.2 (IO2); no longer D5.1 (IO1)
- net USB2_CC2: now also D5.1 (IO1); no longer D5.2 (IO2)

Commit message: nRF wiring done
Both the wires from the raspberry to the nRF and nRF to gpio wires done.
That leaves only the dac and cleanup.
Other:
- sheet Co processor ports: added +3v3_PI; removed none
Changed lines of the file:
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@@
 	)
 	(junction
+		(at 228.6 22.86)
+		(diameter 0)
+		(color 0 0 0 0)
+	)
+	(junction
 		(at 278.13 115.57)
 		(diameter 0)
@@
 	(wire
 		(pts
-			(xy 154.94 22.86) (xy 274.32 22.86)
+			(xy 154.94 22.86) (xy 228.6 22.86)
 		)
 		(stroke
@@
 	(wire
 		(pts
+			(xy 228.6 22.86) (xy 274.32 22.86)
+		)
+		(stroke
+			(width 0)
+			(type default)
+		)
+	)
+	(wire
+		(pts
 			(xy 248.92 64.77) (xy 248.92 74.93)
 		)
@@
 	(wire
 		(pts
+			(xy 228.6 22.86) (xy 228.6 27.94)
+		)
+		(stroke
+			(width 0)
+			(type default)
+		)
+	)
+	(wire
+		(pts
 			(xy 278.13 19.05) (xy 278.13 115.57)
 		)
@@
 			)
 		)
+		(pin "+3v3_PI" input
+			(at 228.6 27.94 90)
+			(effects
+				(font
+					(size 1.27 1.27)
+				)
+				(justify right)
+			)
+		)

Commit message: Fixing up some DRC errors
Parts:
- removed TP7: TestPoint, TestPoint:TestPoint_Pad_D1.0mm, symbol Connector:TestPoint
Changed lines of the file:
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@@
-	)
-	(junction
-		(at 67.31 38.1)
-		(diameter 0)
-		(color 0 0 0 0)
 	)
 	(junction
@@
 	(wire
 		(pts
-			(xy 67.31 38.1) (xy 83.82 38.1)
-		)
-		(stroke
-			(width 0)
-			(type default)
-		)
-	)
-	(wire
-		(pts
 			(xy 274.32 148.59) (xy 274.32 161.29)
 		)
@@
 	(wire
 		(pts
-			(xy 53.34 38.1) (xy 67.31 38.1)
+			(xy 53.34 38.1) (xy 83.82 38.1)
 		)
 		(stroke
@@
 		)
 	)
-	(symbol
-		(lib_id "Connector:TestPoint")
-		(at 67.31 38.1 0)
-		(unit 1)
-		(body_style 1)
-		(exclude_from_sim no)
-		(in_bom yes)
-		(on_board yes)
-		(in_pos_files yes)
-		(dnp no)
-		(property "Reference" "TP7"
-			(at 66.04 34.544 0)
-			(show_name no)
-			(do_not_autoplace no)
-			(effects
-				(font
-					(size 1.27 1.27)
-				)
-				(justify right)
-			)
-		)
-		(property "Value" "TestPoint"
-			(at 64.77 33.5281 0)
-			(hide yes)
-			(show_name no)
-			(do_not_autoplace no)
-			(effects
-				(font
-					(size 1.27 1.27)
-				)
-				(justify right)
-			)
-		)
-		(property "Footprint" "TestPoint:TestPoint_Pad_D1.0mm"
-			(at 72.39 38.1 0)
-			(hide yes)
-			(show_name no)
-			(do_not_autoplace no)
-			(effects
-				(font
-					(size 1.27 1.27)
-				)
-			)
-		)
-		(property "Datasheet" ""
-			(at 72.39 38.1 0)
-			(hide yes)
-			(show_name no)
-			(do_not_autoplace no)
-			(effects
-				(font
-					(size 1.27 1.27)
-				)
-			)
-		)
-		(property "Description" "test point"
-			(at 67.31 38.1 0)
-			(hide yes)
-			(show_name no)
-			(do_not_autoplace no)
-			(effects
-				(font
-					(size 1.27 1.27)
-				)
-			)
-		)
-		(pin "1"
-		)
-		(instances
-			(project "mainboard"
-				(path "/5b8aa782-5c3d-43e7-a869-3bd000015f52"
-					(reference "TP7")
-					(unit 1)
-				)
-			)
-		)
-	)

Commit message: Fix all non-clearance related DRC violations
The clearance ones will need a little extra attention as they are
getting quite close to the manufacturers tolerances
Connections:
- net +5v: now also J3.3 (Pin_3), J3.4 (Pin_4); no longer J3.1 (Pin_1), J3.2 (Pin_2)
- net GND: now also J3.1 (Pin_1), J3.2 (Pin_2); no longer J3.3 (Pin_3), J3.4 (Pin_4)
Other:
- moved on the sheet: J3
Changed lines of the file:
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@@
 	(symbol
 		(lib_id "Connector:Conn_01x04_Pin")
-		(at 77.47 96.52 270)
+		(at 74.93 96.52 90)
+		(mirror x)
 		(unit 1)
 		(body_style 1)
@@
 		(in_pos_files yes)
 		(dnp no)
-		(fields_autoplaced yes)
 		(property "Reference" "J3"
 			(at 76.2 91.44 90)
@@
 		)
 		(property "Footprint" "Connector_PinHeader_2.54mm:PinHeader_1x04_P2.54mm_Vertical"
-			(at 77.47 96.52 0)
+			(at 74.93 96.52 0)
 			(hide yes)
 			(show_name no)
@@
 		)
 		(property "Datasheet" ""
-			(at 77.47 96.52 0)
+			(at 74.93 96.52 0)
 			(hide yes)
 			(show_name no)
@@
 		)
 		(property "Description" "Generic connector, single row, 01x04, script generated"
-			(at 77.47 96.52 0)
+			(at 74.93 96.52 0)
 			(hide yes)
 			(show_name no)
