File: pcb/v0.1/mainboard.kicad_pcb (KiCad board)
At the start: 4 copper layers, 98.2 x 88.7 mm, 128 parts, among them J1 Conn_01x02_Pin, J11 Conn_01x03_Pin, J12 Conn_02x08_Odd_Even, J13 Conn_02x08_Odd_Even, J2 TYPE_C_Receptacle, J3 Conn_01x04_Pin, J4 TYPE_C_Receptacle, J5 TYPE_C_Receptacle, J6 22s_disp_connector, J7 ComputeModule5-CM5_connector, J8 Micro_SD_molex, J9 AudioJack3, Q1 MMBT2222A, SW1 SW_Push_45deg, U1 AP2112K-3.3TRG1, U2 Nexperia PUSB3FR4Z, U3 Nexperia PUSB3FR4Z, U4 PCM5102A, U5 RT9742GGJ5, U6 RT9742GGJ5, U7 MDBT50Q-P1MV2, U8 AP22653W6-7, Y1 O_32.768kHz

Commit message: No more DRC!
Routing:
- net /+5v: track 329.9 -> 328.6 mm, vias 24 -> 23
Changed lines of the file:
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@@
 		(sheetname "/HighSpeed/")
 		(sheetfile "high_speed.kicad_sch")
-		(units
-			(unit
-				(name "A")
-				(pins "SH" "B1" "B12" "A1" "A12" "B9" "A9" "B4" "A4" "A5" "B5" "A7" "B7"
-					"A6" "B6" "B10" "B11" "A3" "A2" "A10" "A11" "B3" "B2" "A8" "B8"
-				)
-			)
-		)
 		(solder_mask_margin 0)
 		(clearance 0.1)
@@
 		)
 		(pad "" np_thru_hole oval
-			(at 9.03 3.7304 270)
+			(at 9.04 3.7304 270)
 			(size 0.9398 0.6604)
-			(drill oval 0.95 0.6604)
+			(drill oval 0.94 0.6604)
 			(layers "*.Cu" "*.Mask")
 		)
@@
 		(sheetname "/HighSpeed/")
 		(sheetfile "high_speed.kicad_sch")
-		(units
-			(unit
-				(name "A")
-				(pins "SH" "B1" "B12" "A1" "A12" "B9" "A9" "B4" "A4" "A5" "B5" "A7" "B7"
-					"A6" "B6" "B10" "B11" "A3" "A2" "A10" "A11" "B3" "B2" "A8" "B8"
-				)
-			)
-		)
 		(solder_mask_margin 0)
 		(clearance 0.1)
@@
 		)
 		(pad "" np_thru_hole oval
-			(at 9.03 3.7304 270)
+			(at 9.04 3.7304 270)
 			(size 0.9398 0.6604)
-			(drill oval 0.95 0.6604)
+			(drill oval 0.94 0.6604)
 			(layers "*.Cu" "*.Mask")
 		)
@@
 		(sheetname "/")
 		(sheetfile "mainboard.kicad_sch")
-		(units
-			(unit
-				(name "A")
-				(pins "SH" "B1" "B12" "A1" "A12" "B9" "A9" "B4" "A4" "A5" "B5" "A7" "B7"
-					"A6" "B6" "B10" "B11" "A3" "A2" "A10" "A11" "B3" "B2" "A8" "B8"
-				)
-			)
-		)
 		(solder_mask_margin 0)
 		(clearance 0.1)
@@
 		)
 		(pad "" np_thru_hole oval
-			(at 9.03 3.7304 270)
+			(at 9.04 3.7304 270)
 			(size 0.9398 0.6604)
-			(drill oval 0.95 0.6604)
+			(drill oval 0.94 0.6604)
 			(layers "*.Cu" "*.Mask")
 		)
@@
 	)
 	(segment
-		(start 90.390305 51.143031)
-		(end 91.100305 51.143031)
-		(width 0.25)
-		(layer "F.Cu")
-		(net "/+5v")
-	)
-	(segment
 		(start 87.400305 50.142779)
 		(end 87.400305 50.143031)
@@
 	)
 	(via
-		(at 91.100305 51.143031)
-		(size 0.6)
-		(drill 0.3)
-		(layers "F.Cu" "B.Cu")
-		(net "/+5v")
-	)
-	(via
 		(at 84.100305 78.883031)
 		(size 0.6)
@@
 	)
 	(segment
+		(start 90.147274 46.89)
+		(end 88.07 46.89)
+		(width 1)
+		(layer "B.Cu")
+		(net "/+5v")
+	)
+	(segment
 		(start 98.915305 50.668031)
 		(end 94.870305 46.623031)
@@
 	)
 	(segment
+		(start 88.07 46.89)
+		(end 87.85 47.11)
+		(width 1)
+		(layer "B.Cu")
+		(net "/+5v")
+	)
+	(segment
 		(start 152.075305 61.768031)
 		(end 155.100305 64.793031)
@@
 	)
 	(segment
-		(start 90.300305 47.043031)
-		(end 90.700305 47.443031)
-		(width 0.6)
-		(layer "B.Cu")
-		(net "/+5v")
-	)
-	(segment
 		(start 95.36 52.43)
 		(end 94.98 52.43)
@@
 	)
 	(segment
+		(start 90.700305 47.443031)
+		(end 90.147274 46.89)
+		(width 1)
+		(layer "B.Cu")
+		(net "/+5v")
+	)
+	(segment
 		(start 98.890305 57.943031)
 		(end 98.890305 58.578031)
@@
 	)
 	(segment
+		(start 89.967274 50.72)
+		(end 90.390305 51.143031)
+		(width 1)
+		(layer "B.Cu")
+		(net "/+5v")
+	)
+	(segment
 		(start 157.650305 64.793031)
 		(end 157.625305 64.818031)
@@
 	)
 	(segment
+		(start 87.71 50.72)
+		(end 89.967274 50.72)
+		(width 1)
+		(layer "B.Cu")
+		(net "/+5v")
+	)
+	(segment
 		(start 123.325305 61.268031)
 		(end 113.785305 61.268031)
@@
 	)
 	(segment
-		(start 87.500305 50.873031)
-		(end 90.830305 50.873031)
-		(width 0.6)
-		(layer "B.Cu")
-		(net "/+5v")
-	)
-	(segment
 		(start 113.785305 61.268031)
 		(end 108.000305 67.053031)
@@
 		(layer "B.Cu")
 		(net "/+5v")
-	)
-	(segment
-		(start 87.530305 47.043031)
-		(end 90.300305 47.043031)
-		(width 0.6)
-		(layer "B.Cu")
-		(net "/+5v")

Commit message: Fix: USB HS lines having gaps in the reference GND lane.
Routing:
- net GND: vias 431 -> 449
- added copper zone on In2.Cu, net GND
Changed lines of the file:
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@@
 		(capping no)
 		(filling no)
-		(zone_defaults)
 		(pcbplotparams
 			(layerselection 0x00000000_00000000_55555555_5755f5ff)
@@
 	)
 	(via
+		(at 95.62 80.83)
+		(size 0.6)
+		(drill 0.3)
+		(layers "F.Cu" "B.Cu")
+		(free yes)
+		(net "GND")
+	)
+	(via
 		(at 91.450305 109.318031)
 		(size 0.6)
@@
 	)
 	(via
+		(at 93.68 81.91)
+		(size 0.6)
+		(drill 0.3)
+		(layers "F.Cu" "B.Cu")
+		(free yes)
+		(net "GND")
+	)
+	(via
 		(at 96.250305 115.493031)
 		(size 0.6)
@@
 	)
 	(via
+		(at 102.92 91.33)
+		(size 0.6)
+		(drill 0.3)
+		(layers "F.Cu" "B.Cu")
+		(free yes)
+		(net "GND")
+	)
+	(via
 		(at 176.660305 50.293031)
 		(size 0.6)
@@
 	)
 	(via
+		(at 129.56 96.66)
+		(size 0.6)
+		(drill 0.3)
+		(layers "F.Cu" "B.Cu")
+		(free yes)
+		(net "GND")
+	)
+	(via
 		(at 176.7 54.4475)
 		(size 0.6)
@@
 	)
 	(via
+		(at 110.2 98.67)
+		(size 0.6)
+		(drill 0.3)
+		(layers "F.Cu" "B.Cu")
+		(free yes)
+		(net "GND")
+	)
+	(via
 		(at 123.520305 43.563031)
 		(size 0.6)
@@
 	)
 	(via
+		(at 109.64 94.74)
+		(size 0.6)
+		(drill 0.3)
+		(layers "F.Cu" "B.Cu")
+		(free yes)
+		(net "GND")
+	)
+	(via
+		(at 95.35 83.77)
+		(size 0.6)
+		(drill 0.3)
+		(layers "F.Cu" "B.Cu")
+		(free yes)
+		(net "GND")
+	)
+	(via
 		(at 146.565 127.24)
 		(size 0.6)
@@
 	)
 	(via
+		(at 107.14 95.5)
+		(size 0.6)
+		(drill 0.3)
+		(layers "F.Cu" "B.Cu")
+		(free yes)
+		(net "GND")
+	)
+	(via
 		(at 94.350305 103.368031)
 		(size 0.6)
@@
 	)
 	(via
+		(at 111.35 99.82)
+		(size 0.6)
+		(drill 0.3)
+		(layers "F.Cu" "B.Cu")
+		(free yes)
+		(net "GND")
+	)
+	(via
 		(at 115.700305 47.783031)
 		(size 0.6)
@@
 	)
 	(via
-		(at 108.560305 92.193031)
-		(size 0.6)
-		(drill 0.3)
-		(layers "F.Cu" "B.Cu")
-		(free yes)
-		(net "GND")
-	)
-	(via
 		(at 157.900305 114.243031)
 		(size 0.6)
@@
 	)
 	(via
-		(at 98.050305 87.213031)
+		(at 99.42 84.74)
 		(size 0.6)
 		(drill 0.3)
@@
 	)
 	(via
+		(at 103.47 88.77)
+		(size 0.6)
+		(drill 0.3)
+		(layers "F.Cu" "B.Cu")
+		(free yes)
+		(net "GND")
+	)
+	(via
 		(at 121.400305 114.473031)
 		(size 0.6)
@@
 	)
 	(via
+		(at 96.86 85.25)
+		(size 0.6)
+		(drill 0.3)
+		(layers "F.Cu" "B.Cu")
+		(free yes)
+		(net "GND")
+	)
+	(via
 		(at 124.600305 70.093031)
 		(size 0.6)
@@
 	)
 	(via
+		(at 101.89 87.19)
+		(size 0.6)
+		(drill 0.3)
+		(layers "F.Cu" "B.Cu")
+		(free yes)
+		(net "GND")
+	)
+	(via
 		(at 110.480305 108.443031)
 		(size 0.6)
@@
 	)
 	(via
+		(at 92.37 80.73)
+		(size 0.6)
+		(drill 0.3)
+		(layers "F.Cu" "B.Cu")
+		(free yes)
+		(net "GND")
+	)
+	(via
 		(at 80.23241 49.023031)
 		(size 0.6)
@@
 	)
 	(via
+		(at 113.04 97.96)
+		(size 0.6)
+		(drill 0.3)
+		(layers "F.Cu" "B.Cu")
+		(free yes)
+		(net "GND")
+	)
+	(via
 		(at 118.350305 104.043031)
 		(size 0.6)
@@
 	)
 	(via
+		(at 107.17 92.3)
+		(size 0.6)
+		(drill 0.3)
+		(layers "F.Cu" "B.Cu")
+		(free yes)
+		(net "GND")
+	)
+	(via
 		(at 83.0925 127.24)
 		(size 0.6)
@@
 	)
 	(via
+		(at 111.45 96.67)
+		(size 0.6)
+		(drill 0.3)
+		(layers "F.Cu" "B.Cu")
+		(free yes)
+		(net "GND")
+	)
+	(via
 		(at 129.650305 124.593031)
 		(size 0.6)
@@
 	)
 	(via
+		(at 101.47 89.85)
+		(size 0.6)
+		(drill 0.3)
+		(layers "F.Cu" "B.Cu")
+		(free yes)
+		(net "GND")
+	)
+	(via
 		(at 155.970305 60.823031)
 		(size 0.6)
@@
 	)
 	(via
-		(at 101.410305 90.463031)
-		(size 0.6)
-		(drill 0.3)
-		(layers "F.Cu" "B.Cu")
-		(free yes)
-		(net "GND")
-	)
-	(via
 		(at 137.880305 92.093031)
 		(size 0.6)
@@
 	)
 	(via
+		(at 122.35 91.93)
+		(size 0.6)
+		(drill 0.3)
+		(layers "F.Cu" "B.Cu")
+		(free yes)
+		(net "GND")
+	)
+	(via
 		(at 98.102805 40.213031)
 		(size 0.6)
@@
 	)
 	(via
+		(at 108.41 96.81)
+		(size 0.6)
+		(drill 0.3)
+		(layers "F.Cu" "B.Cu")
+		(free yes)
+		(net "GND")
+	)
+	(via
 		(at 173.585305 40.213031)
 		(size 0.6)
@@
 	)
 	(via
+		(at 99.27 87.66)
+		(size 0.6)
+		(drill 0.3)
+		(layers "F.Cu" "B.Cu")
+		(free yes)
+		(net "GND")
+	)
+	(via
 		(at 111.420305 82.193031)
 		(size 0.6)
@@
 	)
 	(zone
+		(net "GND")
+		(layer "In2.Cu")
+		(hatch edge 0.5)
+		(priority 11)
+		(connect_pads yes
+			(clearance 0.2)
+		)
+		(min_thickness 0.25)
+		(fill yes
+			(thermal_gap 0.5)
+			(thermal_bridge_width 0.5)
+			(island_removal_mode 0)
+		)
+		(polygon
+			(pts
+				(xy 120.92 90.5) (xy 122.11 89.37) (xy 131.03 97.95) (xy 129.71 99.36)
+			)
+		)
+	)
+	(zone
 		(net "/+3v3_LDO")
 		(layer "In2.Cu")
@@
 			)
 		)
+	)
+	(zone
+		(net "GND")
+		(layer "In2.Cu")
+		(hatch edge 0.5)
+		(priority 10)
+		(connect_pads yes
+			(clearance 0.2)
+		)
+		(min_thickness 0.25)
+		(fill yes
+			(thermal_gap 0.5)
+			(thermal_bridge_width 0.5)
+			(island_removal_mode 0)
+		)
+		(polygon
+			(pts
+				(xy 112.33 100.71) (xy 92.29 80.47) (xy 87.37 80.15) (xy 87.4 78.45) (xy 93 78.39) (xy 114.14 99.04)
+			)
+		)
